File: Hardware/CoverUI-legacy-LedPanel-HAT/Legacy-LedPanel-HAT/Legacy-LedPanel-HAT-v1.kicad_sch (KiCad schematic)
At the start: 20 parts, among them J1 Conn_02x20_Odd_Even, J10 2mm, J11 2.54mm, J12 Spare LevelShift A0_A1, J13 Spare LS OUT B0_B1, J14 LS OUT S1_S2, J16 I2C, J2 OM_Serial, J3 1.8mm, J4 2mm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

Commit message: HW redesign based on first live tests (new design not tested)
Parts:
- U1: footprint STM32 Pills:YAAJ_BluePill_SWD_1 -> stm32_pills:YAAJ_WeAct_BlackPill_SWD_2
Connections:
- net +5V: now also U1.40 (5V)
- net GND: no longer U1.40 (GND)
- net LED4 - D4: now also U1.27 (PA1); no longer U1.26 (PA1)
- net LED5 - D5: now also U1.26 (PA0); no longer U1.25 (PA0)
- net LED6 - D6: now also U1.30 (PA4); no longer U1.29 (PA4)
- net LED7 - D7: now also U1.32 (PA6); no longer U1.31 (PA6)
- net LED8 - D8: now also U1.34 (PB0); no longer U1.33 (PB0)
- net LED9 - D9: now also U1.36 (PB2); no longer U1.35 (PB10)
- net Pico-RX_STM32-TX: now also U1.28 (PA2); no longer U1.27 (PA2)
- net Pico-TX_STM32-RX: now also U1.29 (PA3); no longer U1.28 (PA3)
- net S1 (button): now also U1.37 (PB10); no longer U1.36 (PB11)
- net S2 (button): now also U1.31 (PA5); no longer U1.30 (PA5)
- net S3 (button): now also U1.33 (PA7); no longer U1.32 (PA7)
- net S5 (button): now also U1.35 (PB1); no longer U1.34 (PB1)
