File: Hardware/CoverUI-legacy-LedPanel-HAT/Legacy-LedPanel-HAT/Legacy-LedPanel-HAT.kicad_sch (KiCad schematic)
At the start: 37 parts, among them J1 Conn_02x20_Odd_Even, J10 2mm, J11 2.54mm, J12 Spare LevelShift A0_A1, J13 Spare LS OUT B0_B1, J14 LS OUT S1_S2, J16 I2C, J2 OM_Serial, J3 1.8mm, J4 2mm, J5 SOUT_to_STM32, J5_STOP1 2.54mm, J6_STOP2 2.54mm, J7 2mm, J8 1.8mm, J9 1.8mm, U1 STM32F401RC blue pill, U2 74LVC4245AD, U3 STM32F401RC blue pill, U4 LSF0108PWJ, U5 LSF0108PWJ, U6 LSF0108PWJ, U7 LSF0108PWJ, U8 STM32F401RC blue pill

Commit message: commit before merge
Parts:
- removed J3, J8: 1.8mm, CustomFootprintLibrary:conn_01x2_1.8mm, symbol Connector_Generic:Conn_01x02
- removed J5: SOUT_to_STM32, Connector_PinHeader_2.54mm:PinHeader_1x02_P2.54mm_Vertical, symbol Connector:Conn_01x02_Pin
- removed J9: 1.8mm, CustomFootprintLibrary:conn_01x9_1.8mm, symbol Connector_Generic:Conn_01x09
- removed JP15: LS GND_or_5V, Connector_PinHeader_2.54mm:PinHeader_1x03_P2.54mm_Vertical, symbol Jumper:Jumper_3_Bridged12
- removed U2: 74LVC4245AD, SOT137-1_NEX, symbol NXP 74LVC4245AD:74LVC4245AD
- added C1: 0.1uF, Capacitor_SMD:C_1206_3216Metric_Pad1.33x1.80mm_HandSolder, symbol Device:C_Polarized
- added J3: Pill Widening, Connector_PinHeader_2.54mm:PinHeader_1x20_P2.54mm_Vertical, symbol Connector:Conn_01x20_Pin
- added J5: 5V out, Connector_PinHeader_2.54mm:PinHeader_1x03_P2.54mm_Vertical, symbol Connector:Conn_01x03_Pin
- added J6: 3V3 out, Connector_PinHeader_2.54mm:PinHeader_1x03_P2.54mm_Vertical, symbol Connector:Conn_01x03_Pin
- added J8: GND out, Connector_PinHeader_2.54mm:PinHeader_1x03_P2.54mm_Vertical, symbol Connector:Conn_01x03_Pin
- added R1: 200k, Resistor_SMD:R_1206_3216Metric_Pad1.30x1.75mm_HandSolder, symbol Device:R
- added U2: LSF0108PWJ, TSSOP20_SOT360-1_NEX, symbol LSF0108PWJ-sequential:LSF0108PWJ
- J10: footprint Connector_JST:JST_PH_S9B-PH-K_1x09_P2.00mm_Horizontal -> Connector_JST:JST_PH_B9B-PH-K_1x09_P2.00mm_Vertical
- J11: footprint Connector_JST:JST_XH_S9B-XH-A-1_1x09_P2.50mm_Horizontal -> Connector_JST:JST_XH_B9B-XH-A_1x09_P2.50mm_Vertical
- J12: value Spare LevelShift A0_A1 -> Spare LevelShift A6-8; footprint Connector_PinHeader_2.54mm:PinHeader_1x02_P2.54mm_Horizontal -> Connector_PinHeader_2.54mm:PinHeader_1x03_P2.54mm_Vertical; symbol Connector:Conn_01x02_Pin -> Connector:Conn_01x03_Pin
- J13: value Spare LS OUT B0_B1 -> Spare LS OUT B6-8; footprint Connector_PinHeader_2.54mm:PinHeader_1x02_P2.54mm_Horizontal -> Connector_PinHeader_2.54mm:PinHeader_1x03_P2.54mm_Vertical; symbol Connector:Conn_01x02_Pin -> Connector:Conn_01x03_Pin
- J14: value LS OUT S1_S2 -> LS OUT S1_S2_SOUT; footprint Connector_PinHeader_2.54mm:PinHeader_1x02_P2.54mm_Horizontal -> Connector_PinHeader_2.54mm:PinHeader_1x03_P2.54mm_Vertical; symbol Connector:Conn_01x02_Pin -> Connector:Conn_01x03_Pin
- J16: footprint Connector_PinHeader_2.54mm:PinHeader_1x02_P2.54mm_Horizontal -> Connector_PinHeader_2.54mm:PinHeader_1x02_P2.54mm_Vertical
- JP7: value STOP1 GND_or_5V -> ESTOP 5V_or_3V3
- JP8: value STOP2 GND_or_5V -> ESTOP1 LS_or_uC
- U1: footprint STM32 Pills:YAAJ_BluePill_SWD_1 -> stm32_pills:YAAJ_WeAct_BlackPill_SWD_2
- renumbered C1 to C2, C2 to C3, C3 to C4, C4 to C5, R1 to R2, R2 to R3, R3 to R4, R4 to R5
Connections:
- net ESTOP2 is gone; now on net JP1-1 Right Bumper: U1.2 (PB13)
- net +5V: now also JP1.3 (B), JP2.1 (A), JP7.1 (A), U1.40 (5V), U3.18 (5V), U3.40 (5V), U4.2 (REFA), U5.2 (REFA), U6.2 (REFA), U7.2 (REFA), U8.18 (5V), U8.40 (5V), J3.18 (Pin_18), J5.1 (Pin_1), J5.2 (Pin_2), J5.3 (Pin_3), U2.2 (REFA); no longer JP7.3 (B), JP8.3 (B)
- net ESTOP1_5V: now also J6_STOP2.2 (Pin_2), J7.2 (Pin_2)
- net ESTOP2_5V: now also JP7.2 (C)
- net GND: now also C1.2, J3.19 (Pin_19), J8.1 (Pin_1), J8.2 (Pin_2), J8.3 (Pin_3), U2.1 (GND); no longer JP7.1 (A), JP8.1 (A)
- net JP1-1 Right Bumper: now also J3.2 (Pin_2); no longer U1.3 (PB14)
- net JP1-10 LiftX: now also U1.6 (PA9), J3.6 (Pin_6); no longer J1.38 (Pin_38), J16.1 (Pin_1), J16.2 (Pin_2), J4.2 (Pin_2), J5_STOP1.2 (Pin_2), U1.14 (PB6), U1.15 (PB7), U1.5 (PA8)
- net JP1-4 Lift: now also U1.3 (PB14), J3.3 (Pin_3); no longer U1.4 (PB15)
- net JP1-7 Left Bumper: now also U1.5 (PA8), J3.5 (Pin_5); no longer U1.6 (PA9)
- net JP5-2 STOP1: now also J3.8 (Pin_8); no longer J6_STOP2.2 (Pin_2), J7.2 (Pin_2)
- net LED10 - D10: now also J3.16 (Pin_16)
- net RAIN: now also U2.17 (B2)
- net RAIN_5V: now also U2.4 (A2)
- net S1 (button): now also J3.13 (Pin_13)
- net S1_5V: now also U2.6 (A4)
- net S1_LS: now also J14.2 (Pin_2), U2.15 (B4); no longer J14.1 (Pin_1)
- net S2 (button): now also J3.17 (Pin_17)
- net S2_5V: now also U2.5 (A3)
- net S2_LS: now also J14.1 (Pin_1), U2.16 (B3); no longer J14.2 (Pin_2)
- net S4 (button): now also J3.9 (Pin_9)
- net S6 (button): now also J3.7 (Pin_7)
- net S7 (button): now also J3.12 (Pin_12)
- net S8 (button): now also J3.10 (Pin_10)
- net S9 (button): now also J3.11 (Pin_11)
- net SOUT_5V: now also U2.7 (A5)
- net SOUT_LS: now also J14.3 (Pin_3), U2.14 (B5)
- net at J6_STOP2.1 (Pin_1), J7.1 (Pin_1): now also J4.2 (Pin_2), J5_STOP1.2 (Pin_2); no longer JP8.2 (C)
- net 3V3: now reaches JP1.1 (A), U1.38 (3V3)
- net 3V3: now also JP2.3 (B), JP7.3 (B), U1.20 (3V3), J3.20 (Pin_20), J6.1 (Pin_1), J6.2 (Pin_2), J6.3 (Pin_3), R1.2
- net at J4.1 (Pin_1), J5_STOP1.1 (Pin_1): now also JP8.2 (C); no longer JP7.2 (C)
- net at J12.1 (Pin_1): now also U2.8 (A6)
- net at J12.2 (Pin_2): now also U2.9 (A7)
- net at J13.2 (Pin_2): now also U2.12 (B7)
- net at J13.1 (Pin_1): now also U2.13 (B6)
- net ESTOP1 renamed ESTOP
- net ESTOP: now also JP8.3 (B), J3.1 (Pin_1), U2.18 (B1)
- new net: J12.3 (Pin_3), U2.10 (A8)
- new net: C1.1, R1.1, U2.19 (REFB), U2.20 (EN)
- new net: J13.3 (Pin_3), U2.11 (B8)
- new net ESTOP_5V: JP8.1 (A), U2.3 (A1)
- new net JP6-2 STOP2: J1.38 (Pin_38), J3.4 (Pin_4), U1.4 (PB15)
- new net SCL1: J16.1 (Pin_1), J3.14 (Pin_14), U1.14 (PB6)
- new net SDA1: J16.2 (Pin_2), J3.15 (Pin_15), U1.15 (PB7)
Other:
- moved on the sheet: J4, J5_STOP1, J6_STOP2, J7, JP7, JP8

Commit message: HW redesign based on first live tests (new design not tested)
Parts:
- removed C1, C2, C3, C4, C5: 0.1uF, Capacitor_SMD:C_1206_3216Metric_Pad1.33x1.80mm_HandSolder, symbol Device:C_Polarized
- removed J12: Spare LevelShift A6-8, Connector_PinHeader_2.54mm:PinHeader_1x03_P2.54mm_Vertical, symbol Connector:Conn_01x03_Pin
- removed J13: Spare LS OUT B6-8, Connector_PinHeader_2.54mm:PinHeader_1x03_P2.54mm_Vertical, symbol Connector:Conn_01x03_Pin
- removed J14: LS OUT S1_S2_SOUT, Connector_PinHeader_2.54mm:PinHeader_1x03_P2.54mm_Vertical, symbol Connector:Conn_01x03_Pin
- removed J16: I2C, Connector_PinHeader_2.54mm:PinHeader_1x02_P2.54mm_Vertical, symbol Connector:Conn_01x02_Pin
- removed J4: 2mm, Connector_JST:JST_PH_B2B-PH-K_1x02_P2.00mm_Vertical, symbol Connector_Generic:Conn_01x02
- removed JP7: ESTOP 5V_or_3V3, Connector_PinHeader_2.54mm:PinHeader_1x03_P2.54mm_Vertical, symbol Jumper:Jumper_3_Bridged12
- removed JP8: ESTOP1 LS_or_uC, Connector_PinHeader_2.54mm:PinHeader_1x03_P2.54mm_Vertical, symbol Jumper:Jumper_3_Bridged12
- removed R2, R3, R4, R5: 200k, Resistor_SMD:R_1206_3216Metric_Pad1.30x1.75mm_HandSolder, symbol Device:R
- removed U2, U4, U5, U6, U7: LSF0108PWJ, TSSOP20_SOT360-1_NEX, symbol LSF0108PWJ-sequential:LSF0108PWJ
- removed U3, U8: STM32F401RC blue pill, STM32 Pills:YAAJ_BluePill_1, symbol YAAJ_BluePill_SWD_Breakout:YAAJ_BluePill_SWD_Breakout
- added C1: 100nF, Capacitor_SMD:C_1812_4532Metric, symbol Device:C
- added D1: PDZ3.3B.115, Diode_SMD:D_1812_4532Metric, symbol Device:D_Zener
- added J12: 2mm, Connector_JST:JST_PH_B2B-PH-K_1x02_P2.00mm_Vertical, symbol Connector_Generic:Conn_01x02
- added J4: SWO, Connector_PinHeader_2.54mm:PinHeader_1x01_P2.54mm_Vertical, symbol Connector:Conn_01x01_Pin
- R1: value 200k -> 10k; footprint Resistor_SMD:R_1206_3216Metric_Pad1.30x1.75mm_HandSolder -> Resistor_SMD:R_1812_4532Metric_Pad1.30x3.40mm_HandSolder
- renumbered J7 to J13
Connections:
- net +5V: now also J3.20 (Pin_20); no longer J3.18 (Pin_18)
- net 3V3: now also J3.18 (Pin_18); no longer J3.20 (Pin_20), R1.2
- net GND: now also J13.1 (Pin_1), J5_STOP1.1 (Pin_1), J6_STOP2.1 (Pin_1), C1.2, D1.2 (A), J12.1 (Pin_1); no longer J10.6 (Pin_6), J11.6 (Pin_6)
- net JP1-1 Right Bumper: now also U1.4 (PB15); no longer J3.2 (Pin_2), U1.2 (PB13)
- net JP1-10 LiftX: now also U1.7 (PA10); no longer J3.6 (Pin_6), U1.6 (PA9)
- net JP1-4 Lift: no longer J3.3 (Pin_3)
- net JP1-7 Left Bumper: now also U1.9 (PA12); no longer J3.5 (Pin_5), U1.5 (PA8)
- net JP5-2 STOP1: now also J5_STOP1.2 (Pin_2), U1.6 (PA9), J12.2 (Pin_2); no longer J3.8 (Pin_8), U1.8 (PA11)
- net JP6-2 STOP2: now also J13.2 (Pin_2), J6_STOP2.2 (Pin_2), U1.5 (PA8); no longer J3.4 (Pin_4), U1.4 (PB15)
- net LED1 - D1: now also J3.2 (Pin_2)
- net LED10 - D10: now also U1.36 (PB2); no longer U1.16 (PB8)
- net LED2 - D2: now also J3.4 (Pin_4)
- net LED3 - D3: now also J3.3 (Pin_3)
- net LED4 - D4: now also J3.7 (Pin_7)
- net LED5 - D5: now also J3.6 (Pin_6)
- net LED6 - D6: now also J3.10 (Pin_10)
- net LED7 - D7: now also J3.11 (Pin_11)
- net LED8 - D8: now also J3.13 (Pin_13)
- net LED9 - D9: now also U1.16 (PB8); no longer U1.36 (PB2)
- net Pico-RX_STM32-TX: now also J3.8 (Pin_8)
- net Pico-TX_STM32-RX: now also J3.9 (Pin_9)
- net RAIN: now also J3.15 (Pin_15), R1.2
- net RAIN_5V: now also R1.1, C1.1, D1.1 (K)
- net S1 (button): now also U1.15 (PB7); no longer J3.13 (Pin_13), U1.13 (PB5)
- net S2 (button): no longer J3.17 (Pin_17)
- net S3 (button): now also J3.12 (Pin_12)
- net S4 (button): now also U1.10 (PA15); no longer J3.9 (Pin_9), U1.9 (PA12)
- net S5 (button): now also J3.14 (Pin_14)
- net S6 (button): now also U1.8 (PA11); no longer J3.7 (Pin_7), U1.7 (PA10)
- net S7 (button): now also U1.14 (PB6); no longer J3.12 (Pin_12), U1.12 (PB4)
- net S8 (button): now also U1.13 (PB5); no longer J3.10 (Pin_10), U1.10 (PA15)
- net S9 (button): now also U1.12 (PB4); no longer J3.11 (Pin_11), U1.11 (PB3)
- net at U1.21 (VBat): now also J3.1 (Pin_1)
- net at U1.25 (RST): now also J3.5 (Pin_5)
- net ESTOP renamed ESTOP1
- net ESTOP1: now also J10.8 (Pin_8), J11.8 (Pin_8); no longer J3.1 (Pin_1)
- removed net ESTOP1_5V: J10.8 (Pin_8), J11.8 (Pin_8), J13.2 (Pin_2), J6_STOP2.2 (Pin_2)
- net ESTOP2_5V renamed ESTOP2
- net ESTOP2: now also U1.2 (PB13)
- net LED11 - D11 renamed LED11 - D11 (S2 LED)
- net LED11 - D11 (S2 LED): now also J3.17 (Pin_17)
- removed net SCL1: J3.14 (Pin_14), U1.14 (PB6)
- removed net SDA1: J3.15 (Pin_15), U1.15 (PB7)
- new net: J4.1 (Pin_1), U1.11 (PB3)
- new net GAIN: J10.6 (Pin_6), J11.6 (Pin_6)
Other:
- moved on the sheet: J13, J2, J3, J5_STOP1, J6_STOP2
